File: Hardware/ARTIC_R2.brd (EAGLE design)
At the start: 22.9 x 50.8 mm, 132 parts, among them J1 U.FL, J2 THING_PLUS, Q1 20V/4.2A/52mΩ/1.4W, U1 32M SPI Flash, U2 1.8V/100mA, U3 ARTIC_R2, U4 RFPA0133, U5 AS179-92LF, U6 DUAL-OPTOISOLATOR_SOIC8, X1 CRYSTAL-TCXO-26MHZ

Commit message: Updated the flash memory
Parts:
- U1: value 32M SPI Flash -> 2Mbit SPI Flash; device SparkFun-IC-Memory:SO08 -> New_Parts_IC-Memory:SO08
Changed lines of the file:
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@@
 <attribute name="PROD_ID" value="RES-13495" x="11.43" y="7.62" size="1.778" layer="27" ratio="15" display="off"/>
-</element>
-<element name="U1" library="SparkFun-IC-Memory" package="SO08" value="32M SPI Flash" x="17.145" y="13.97" smashed="yes">
-<attribute name="NAME" x="17.145" y="14.2875" size="0.6096" layer="25" font="vector" ratio="20" rot="R180" align="bottom-center"/>
-<attribute name="PROD_ID" value="N/A" x="17.145" y="13.97" size="1.778" layer="27" ratio="15" display="off"/>
 </element>
 <element name="C1" library="SparkFun-Capacitors" package="0402-TIGHT" value="10uF" x="13.97" y="8.3185" smashed="yes" rot="R270">
@@
 <attribute name="NAME" x="5.588" y="46.99" size="0.6096" layer="26" font="vector" ratio="20" rot="MR270" align="bottom-center"/>
 </element>
+<element name="U1" library="New_Parts_IC-Memory" package="SO08" value="2Mbit SPI Flash" x="17.145" y="13.97" smashed="yes">
+<attribute name="DIGIKEY_PART" value=" SST25VF020B-80-4I-SAE-TCT-ND" x="17.145" y="13.97" size="1.778" layer="27" ratio="15" display="off"/>
+<attribute name="MANUFACTURER" value="Microchip" x="17.145" y="13.97" size="1.778" layer="27" ratio="15" display="off"/>
+<attribute name="MANU_PART" value="SST25VF020B-80-4I-SAE-T" x="17.145" y="13.97" size="1.778" layer="27" ratio="15" display="off"/>
+<attribute name="MOUSER_PART" value="579-25VF020B8ISAET" x="17.145" y="13.97" size="1.778" layer="27" ratio="15" display="off"/>
+<attribute name="NAME" x="13.97" y="13.97" size="0.6096" layer="25" font="vector" ratio="20" rot="R90" align="bottom-center"/>
+<attribute name="PROD_ID" value="" x="17.145" y="13.97" size="1.778" layer="27" ratio="15" display="off"/>
+<attribute name="VALUE" x="20.955" y="13.97" size="0.6096" layer="27" font="vector" ratio="20" rot="R90" align="bottom-center"/>
+</element>
 </elements>
 <signals>
@@
 <contactref element="C1" pad="2"/>
 <contactref element="J2" pad="25"/>
-<contactref element="U1" pad="4"/>
 <contactref element="C2" pad="2"/>
 <contactref element="C45" pad="2"/>
@@
 <wire x1="2.5908" y1="22.9997" x2="2.5908" y2="28.2448" width="0.254" layer="1"/>
 <via x="2.54" y="45.72" extent="1-16" drill="0.2"/>
+<contactref element="U1" pad="4"/>
 </signal>
 <signal name="EDAP">
@@
 <signal name="FLSH_SCLK">
 <contactref element="U3" pad="12"/>
+<wire x1="16.862" y1="19.333" x2="15.958" y2="19.333" width="0.254" layer="1"/>
+<wire x1="17.78" y1="18.415" x2="16.862" y2="19.333" width="0.254" layer="1"/>
 <contactref element="U1" pad="6"/>
 <wire x1="17.78" y1="16.77" x2="17.78" y2="18.415" width="0.254" layer="1"/>
-<wire x1="16.862" y1="19.333" x2="15.958" y2="19.333" width="0.254" layer="1"/>
-<wire x1="17.78" y1="18.415" x2="16.862" y2="19.333" width="0.254" layer="1"/>
 </signal>
 <signal name="FLSH_SI">
 <contactref element="U3" pad="13"/>
+<wire x1="17.1645" y1="19.983" x2="16.608" y2="19.983" width="0.254" layer="1"/>
+<wire x1="19.05" y1="18.0975" x2="17.1645" y2="19.983" width="0.254" layer="1"/>
 <contactref element="U1" pad="5"/>
 <wire x1="19.05" y1="16.77" x2="19.05" y2="18.0975" width="0.254" layer="1"/>
-<wire x1="17.1645" y1="19.983" x2="16.608" y2="19.983" width="0.254" layer="1"/>
-<wire x1="19.05" y1="18.0975" x2="17.1645" y2="19.983" width="0.254" layer="1"/>
 </signal>
 <signal name="FLSH_SO">
 <contactref element="U3" pad="14"/>
-<contactref element="U1" pad="2"/>
 <via x="16.51" y="12.3825" extent="1-16" drill="0.2"/>
 <wire x1="16.51" y1="12.3825" x2="15.6845" y2="13.208" width="0.254" layer="16"/>
@@
 <wire x1="17.526" y1="20.447" x2="16.644" y2="20.447" width="0.254" layer="1"/>
 <wire x1="16.644" y1="20.447" x2="16.608" y2="20.483" width="0.254" layer="1"/>
-<wire x1="16.51" y1="11.17" x2="16.51" y2="12.3825" width="0.254" layer="1"/>
 <wire x1="15.6845" y1="13.208" x2="15.6845" y2="18.6055" width="0.254" layer="16"/>
 <wire x1="15.6845" y1="18.6055" x2="17.526" y2="20.447" width="0.254" layer="16"/>
+<contactref element="U1" pad="2"/>
+<wire x1="16.51" y1="11.17" x2="16.51" y2="12.3825" width="0.254" layer="1"/>
 </signal>
 <signal name="FLSH_CEN">
 <contactref element="U3" pad="15"/>
-<contactref element="U1" pad="1"/>
-<wire x1="15.24" y1="11.17" x2="15.24" y2="12.3825" width="0.254" layer="1"/>
 <via x="15.24" y="12.3825" extent="1-16" drill="0.2"/>
 <wire x1="15.24" y1="12.3825" x2="15.24" y2="18.796" width="0.254" layer="16"/>
@@
 <wire x1="17.399" y1="20.955" x2="17.371" y2="20.983" width="0.254" layer="1"/>
 <wire x1="17.371" y1="20.983" x2="16.608" y2="20.983" width="0.254" layer="1"/>
+<contactref element="U1" pad="1"/>
+<wire x1="15.24" y1="11.17" x2="15.24" y2="12.3825" width="0.254" layer="1"/>
 </signal>
 <signal name="SCLK">
@@
 <contactref element="C2" pad="1"/>
 <contactref element="L1" pad="1"/>
-<contactref element="U1" pad="8"/>
 <contactref element="R2" pad="2"/>
 <contactref element="R11" pad="2"/>
 <contactref element="C45" pad="1"/>
-<wire x1="15.24" y1="16.77" x2="15.24" y2="15.8115" width="0.254" layer="1"/>
 <wire x1="14.724" y1="15.2955" x2="13.335" y2="15.2955" width="0.254" layer="1"/>
 <wire x1="15.24" y1="15.8115" x2="14.724" y2="15.2955" width="0.254" layer="1"/>
@@
 <wire x1="12.2475" y1="12.8905" x2="13.0255" y2="12.8905" width="0.254" layer="1"/>
 <wire x1="13.0255" y1="12.8905" x2="13.335" y2="13.2" width="0.254" layer="1"/>
+<contactref element="U1" pad="8"/>
+<wire x1="15.24" y1="16.77" x2="15.24" y2="15.8115" width="0.254" layer="1"/>
 </signal>
 <signal name="N$2">
-<contactref element="U1" pad="7"/>
 <contactref element="R2" pad="1"/>
 <wire x1="13.335" y1="14.2955" x2="14.994" y2="14.2955" width="0.254" layer="1"/>
-<wire x1="16.51" y1="15.8115" x2="16.51" y2="16.77" width="0.254" layer="1"/>
-<wire x1="14.994" y1="14.2955" x2="16.51" y2="15.8115" width="0.254" layer="1"/>
+<wire x1="16.51" y1="15.8115" x2="14.994" y2="14.2955" width="0.254" layer="1"/>
+<contactref element="U1" pad="7"/>
+<wire x1="16.51" y1="16.77" x2="16.51" y2="15.8115" width="0.254" layer="1"/>
 </signal>
 <signal name="N$3">
-<contactref element="U1" pad="3"/>
 <contactref element="R11" pad="1"/>
 <wire x1="14.6685" y1="12.835" x2="14.0335" y2="12.2" width="0.254" layer="1"/>
 <wire x1="13.335" y1="12.2" x2="14.0335" y2="12.2" width="0.254" layer="1"/>
 <wire x1="17.264" y1="12.835" x2="14.6685" y2="12.835" width="0.254" layer="1"/>
-<wire x1="17.78" y1="12.319" x2="17.78" y2="11.17" width="0.254" layer="1"/>
-<wire x1="17.264" y1="12.835" x2="17.78" y2="12.319" width="0.254" layer="1"/>
+<wire x1="17.78" y1="12.319" x2="17.264" y2="12.835" width="0.254" layer="1"/>
+<contactref element="U1" pad="3"/>
+<wire x1="17.78" y1="11.17" x2="17.78" y2="12.319" width="0.254" layer="1"/>
 </signal>
 <signal name="N$4">
