File: Hardware/ARTIC_R2.brd (EAGLE design)
At the start: 22.9 x 50.8 mm, 144 parts, among them J1 U.FL, J2 THING_PLUS, J5 Flash Programming, K1 TLP3475R, Q1 3.1A/30V/105mΩ, U1 2Mbit SPI Flash, U2 1.8V/100mA, U3 ARTIC_R2, U4 RFPA0133, U5 AS179-92LF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

Commit message: Update Eagle files - remove New_Parts.lbr
Parts:
- C28: device New_Parts_Capacitors:0402-TIGHT -> SparkFun-Capacitors:0402-TIGHT
- K1: device New_Parts_DiscreteSemi:TLP3475RTPF -> SparkFun-DiscreteSemi:TLP3475RTPF
- L11, L12, L5, L6, L7, L8: device New_Parts_Coils:0402_COILCRAFT -> SparkFun-Coils:0402_COILCRAFT
- R14, R17: device New_Parts_Resistors:0402-TIGHT -> SparkFun-Resistors:0402-TIGHT
- R3: value 3.9OHM -> 3.9; device New_Parts_Resistors:0402-TIGHT -> SparkFun-Resistors:0402-TIGHT
- R6: value 220OHM -> 220; device New_Parts_Resistors:0402-TIGHT -> SparkFun-Resistors:0402-TIGHT
- U1: device New_Parts_IC-Memory:SO08 -> SparkFun-IC-Memory:SO08
- U3: device New_Parts_IC-Comms:QFN-48 -> SparkFun-RF:QFN-48
- U4: device New_Parts_IC-Comms:QFN50P300X300X86-17N -> SparkFun-RF:QFN50P300X300X86-17N
- U5: device New_Parts_IC-Comms:SOT65P220X100-6N -> SparkFun-RF:SOT65P220X100-6N
- U6: device New_Parts_IC-Power:SOT23-5 -> SparkFun-IC-Power:SOT23-5
- X1: device New_Parts_Clocks:CRYSTAL-TCXO-SMD-1.65X1.25 -> SparkFun-Clocks:CRYSTAL-TCXO-SMD-1.65X1.25
